File: pcb/blood_pressure.kicad_pcb (KiCad board)
At the start: 2 copper layers, 68 x 85.5 mm, 18 parts, among them J1 Barrel_Jack, Q1 PMOS, SW1 SW_Push, SW2 SW_SPST, U1 PicoW, U2 3073

Commit message: Final
Parts:
- R4, R5, R6: value 330 -> 60
- moved D2 0.50 mm to (165.5, 82.5)
Routing:
- net VSYS: track 111.5 -> 101.3 mm
- net VBUS: track 101.8 -> 111.3 mm
- net Net-(D1-A): track 79.9 -> 82.6 mm
- net Net-(D2-A): track 62.4 -> 64.3 mm
Other:
- copper layers 2 -> 4

Commit message: Read Me Files
Parts:
- Q1: value PMOS -> DMG2305UX-7; footprint Package_TO_SOT_SMD:SOT-23 -> DMG2305UX_7:SOT91P240X110-3N_DMG2305UX-7
- moved Q1 0.66 mm to (157.5, 50.0)
Connections:
- Q1 pad 1: Net-(Q1-D) -> VBUS
- Q1 pad 2: VBUS -> VSYS
- Q1 pad 3: VSYS -> Net-(SW2-B)
- SW2 pad 2: Net-(Q1-D) -> Net-(SW2-B)
Routing:
- net VBUS: track 111.3 -> 96.4 mm
- net Net-(Q1-D): track 6.77 -> 0.00 mm
- net Net-(SW2-B): track 0.00 -> 4.89 mm
- net VSYS: track 101.3 -> 100.0 mm
